Commit message: update

File: trolley_description/urdf/3d_lidar.xacro (robot description, xacro)
@@ -21,36 +21,4 @@
         </inertial>
     </link>
-    <joint name="2d_lidar_to_body_joint" type="fixed">
-        <parent link = "body" />
-        <child link = "2d_lidar_link" />
-        <origin xyz="0.4 0 0.32" rpy="0 0 0" />   <!--Raised by 0.02 to prevent body link blocking lidar-->
-    </joint>
-    <gazebo reference="2d_lidar_link">
-        <material>Gazebo/Red</material>
-        <sensor name="laser" type="ray">
-            <pose> 0 0 0 0 0 0 </pose>
-            <visualize>true</visualize>
-            <update_rate>20</update_rate>
-            <ray>
-                <scan>
-                    <horizontal>
-                        <samples>360</samples>
-                        <min_angle>-3.14</min_angle>
-                        <max_angle>3.14</max_angle>
-                    </horizontal>
-                </scan>
-                <range>
-                    <min>0</min>
-                    <max>10</max>
-                </range>
-            </ray>
-            <plugin name="laser_controller" filename="libgazebo_ros_ray_sensor.so">
-                <ros>
-                    <argument>~/out:=scan</argument>  <!--Throws warning, that the syntax is deprecated. But our ros2 version is not consistent with newer syntax. So just ignore warning.-->
-                </ros>
-                <output_type>sensor_msgs/LaserScan</output_type>
-                <frame_name>2d_lidar_link</frame_name>
-            </plugin>
-        </sensor>
-    </gazebo>
+    <!--INCOMPLETE-->
 </robot>

Commit message: Update(3d lidar)

File: trolley_description/urdf/3d_lidar.xacro (robot description, xacro)
@@ -3,22 +3,59 @@
     <link name="3d_lidar_link">
         <visual>
-            <origin xyz="0 0 0.015" rpy="0 0 0" />
+            <origin xyz="0 0 0" rpy="0 0 0" />
             <geometry>
-                <cylinder radius="0.05" length="0.03"/>
+                <cylinder radius="0.02" length="0.02"/>
             </geometry>
-            <material name="grey" />
         </visual>
         <collision>
-            <origin xyz="0 0 0.06" rpy="0 0 0" />
+            <origin xyz="0 0 0" rpy="0 0 0" />
             <geometry>
-                <cylinder radius="0.08" length="0.09"/>
+                <cylinder radius="0.01" length="0.01"/>
             </geometry>
         </collision>
         <inertial>
-            <origin xyz="0 0 0.06" rpy="0 0 0" />
+            <origin xyz="0 0 0" rpy="0 0 0" />
             <mass value="0.2"/>
             <inertia ixx="0.000455" ixy="0" ixz="0" iyy="0.000455" iyz="0" izz="0.00064"/>
         </inertial>
     </link>
-    <!--INCOMPLETE-->
+    <joint name="3d_lidar_to_body_joint" type="fixed">
+        <parent link = "body" />
+        <child link = "3d_lidar_link" />
+        <origin xyz="0.45 0 0.415" rpy="0 0 0" />    <!--have put x=0.45 instead of 0.41, just for debugging-->
+    </joint>
+    <!--############################-->
+    <gazebo reference="3d_lidar_link">
+        <sensor name="lidar_3d" type="ray">
+            <pose>0 0 0 0 0 0</pose>
+            <visualize>true</visualize>
+            <update_rate>20</update_rate>
+            <ray>
+                <scan>
+                    <horizontal>
+                        <samples>180</samples>
+                        <min_angle>-1.57</min_angle>
+                        <max_angle>1.57</max_angle>
+                    </horizontal>
+                    <vertical>
+                        <samples>270</samples>
+                        <min_angle>-1.57</min_angle>
+                        <max_angle>3.14</max_angle>
+                    </vertical>
+                </scan>
+                <range>
+                    <min>0.116</min>
+                    <max>10.0</max>
+                    <resolution>0.01</resolution>
+                </range>
+            </ray>
+            <plugin name="lidar_plugin_3d" filename="libgazebo_ros_ray_sensor.so">
+            <ros>
+                <argument>~/out:=/velodyne_points</argument>
+            </ros>
+            <frame_name>3d_lidar_link</frame_name>
+            <output_type>sensor_msgs/PointCloud2</output_type>
+            </plugin>
+        </sensor>
+    </gazebo>
 </robot>

File: trolley_description/urdf/links_joints.xacro (robot description, xacro)
@@ -8,5 +8,5 @@
                 <box size="0.8 0.4 0.3" />
             </geometry>
-            <material name="red" />
+            <material name="blue" />
         </visual>
         <collision>

File: trolley_description/urdf/materials.xacro (robot description, xacro)
@@ -7,3 +7,6 @@
         <color rgba="0.8 0.8 0.8 1" />
     </material>
+    <material name="blue">
+        <color rgba="0 0 0.8 1" />
+    </material>
 </robot>

File: trolley_description/urdf/trolley_urdf.xacro (robot description, xacro)
@@ -5,5 +5,6 @@
     <xacro:include filename="colors.xacro"/>
     <xacro:include filename="diff_drive_plugin.xacro"/>
-    <xacro:include filename="camera.xacro"/>
-    <xacro:include filename="2d_lidar.xacro"/>
+    <!--<xacro:include filename="camera.xacro"/>-->
+    <!--<xacro:include filename="2d_lidar.xacro"/>-->
+    <xacro:include filename="3d_lidar.xacro"/>
 </robot>
